File: kicad/model_train_controller/model_train_controller.kicad_pcb (KiCad board)
At the start: 2 copper layers, 84 x 84 mm, 31 parts, among them J1 LED, J2 ST_BLA, J3 Barrel_Jack_Switch, J5 Conn_02x06_Odd_Even, J6 ST_BLA, Q1 AOSP36326C, Q2 AOSP36326C, Q3 AOSP36326C, Q5 AOSP36326C

Commit message: updated PBC Files and BOM
Parts:
- J1: footprint Connector_PinHeader_2.54mm:PinHeader_1x04_P2.54mm_Vertical -> TerminalBlock_Phoenix:TerminalBlock_Phoenix_MPT-0,5-4-2.54_1x04_P2.54mm_Horizontal; moved to B.Cu
- J2: moved to F.Cu
- moved J1 7.66 mm to (85.0, 89.8), turned to 90 degrees
- moved J2 3.50 mm to (101.8, 127.7), turned to 180 degrees
Connections:
- J1 pad 1: +5V -> GND
- J1 pad 2: /CLK -> /DATA
- J1 pad 3: /DATA -> /CLK
- J1 pad 4: GND -> +5V
- J2 pad 1: /COIL -> +5V
- J2 pad 2: +5V -> /COIL
Other:
- board text added: "CLK"
- board text added: "DATA"
- board text added: "LED STRIP"
- board text added: "Use Screw Terminal If Connecting DC Motor"
- board text added: "WIRELESS LED COIL"
