File: kicad/model_train_controller/model_train_controller.kicad_sch (KiCad schematic)
At the start: 27 parts, among them J1 LED, J2 ST_BLA, J3 Barrel_Jack_Switch, J5 Conn_02x06_Odd_Even, J6 ST_BLA, Q1 AOSP36326C, Q2 AOSP36326C, Q3 AOSP36326C, Q5 AOSP36326C

Commit message: updated PBC Files and BOM
Parts:
- J1: footprint Connector_PinHeader_2.54mm:PinHeader_1x04_P2.54mm_Vertical -> TerminalBlock_Phoenix:TerminalBlock_Phoenix_MPT-0,5-4-2.54_1x04_P2.54mm_Horizontal
Connections:
- net +5V: now also J1.4 (Pin_4), J2.1 (Pin_1); no longer J1.1 (Pin_1), J2.2 (Pin_2)
- net CLK: now also J1.3 (Pin_3); no longer J1.2 (Pin_2)
- net COIL: now also J2.2 (Pin_2); no longer J2.1 (Pin_1)
- net DATA: now also J1.2 (Pin_2); no longer J1.3 (Pin_3)
- net GND: now also J1.1 (Pin_1); no longer J1.4 (Pin_4)
Changed lines of the file:
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@@
 	(symbol
 		(lib_id "Connector:Screw_Terminal_01x02")
-		(at 245.11 133.35 0)
-		(unit 1)
-		(exclude_from_sim no)
-		(in_bom yes)
-		(on_board yes)
-		(dnp no)
-		(fields_autoplaced yes)
+		(at 245.11 135.89 0)
+		(mirror x)
+		(unit 1)
+		(exclude_from_sim no)
+		(in_bom yes)
+		(on_board yes)
+		(dnp no)
 		(property "Reference" "J2"
+			(at 248.285 135.89 0)
+			(effects
+				(font
+					(size 1.27 1.27)
+				)
+				(justify left)
+			)
+		)
+		(property "Value" "ST_BLA"
 			(at 248.285 133.35 0)
 			(effects
@@
 			)
 		)
-		(property "Value" "ST_BLA"
-			(at 248.285 135.89 0)
-			(effects
-				(font
-					(size 1.27 1.27)
-				)
-				(justify left)
-			)
-		)
 		(property "Footprint" "TerminalBlock_Phoenix:TerminalBlock_Phoenix_PT-1,5-2-3.5-H_1x02_P3.50mm_Horizontal"
-			(at 245.11 133.35 0)
+			(at 245.11 135.89 0)
 			(effects
 				(font
@@
 		)
 		(property "Datasheet" "~"
-			(at 245.11 133.35 0)
+			(at 245.11 135.89 0)
 			(effects
 				(font
@@
 		)
 		(property "Description" ""
-			(at 245.11 133.35 0)
+			(at 245.11 135.89 0)
 			(effects
 				(font
@@
 		)
 		(property "Digikey Part No." "277-5719-ND"
-			(at 245.11 133.35 0)
+			(at 245.11 135.89 0)
 			(effects
 				(font
@@
 	(symbol
 		(lib_id "Connector_Generic:Conn_01x04")
-		(at 109.22 139.7 0)
-		(unit 1)
-		(exclude_from_sim no)
-		(in_bom yes)
-		(on_board yes)
-		(dnp no)
-		(fields_autoplaced yes)
+		(at 109.22 142.24 0)
+		(mirror x)
+		(unit 1)
+		(exclude_from_sim no)
+		(in_bom yes)
+		(on_board yes)
+		(dnp no)
 		(property "Reference" "J1"
-			(at 111.76 139.6999 0)
+			(at 111.76 142.2401 0)
 			(effects
 				(font
@@
 		)
 		(property "Value" "LED"
-			(at 111.76 142.2399 0)
+			(at 111.76 139.7001 0)
 			(effects
 				(font
@@
 			)
 		)
-		(property "Footprint" "Connector_PinHeader_2.54mm:PinHeader_1x04_P2.54mm_Vertical"
-			(at 109.22 139.7 0)
+		(property "Footprint" "TerminalBlock_Phoenix:TerminalBlock_Phoenix_MPT-0,5-4-2.54_1x04_P2.54mm_Horizontal"
+			(at 109.22 142.24 0)
 			(effects
 				(font
@@
 		)
 		(property "Datasheet" "~"
-			(at 109.22 139.7 0)
+			(at 109.22 142.24 0)
 			(effects
 				(font
@@
 		)
 		(property "Description" "Generic connector, single row, 01x04, script generated (kicad-library-utils/schlib/autogen/connector/)"
-			(at 109.22 139.7 0)
+			(at 109.22 142.24 0)
 			(effects
 				(font
@@
 		)
 		(property "Digikey Part No." "732-691210910004-ND"
-			(at 109.22 139.7 0)
-			(effects
-				(font
+			(at 109.22 142.24 0)
+			(effects
+				(font
